File: pcbs/right/right.kicad_pcb (KiCad board)
At the start: 2 copper layers, 135.8 x 108.4 mm, 70 parts

Commit message: added fill
Routing:
- added copper zone on B.Cu, net (none)
- added copper zone on F.Cu, net (none)
