File: GLP/ergogen/output/pcbs/left.kicad_pcb (KiCad board)
At the start: 2 copper layers, 138.8 x 106.7 mm, 66 parts

Commit message: ok
Parts:
- added H1: , ceoloide:mounting_hole_plated, F.Cu at (160.0, 106.5)
- added H2: , ceoloide:mounting_hole_plated, F.Cu at (175.0, 106.5)
- moved D28 15.4 mm to (168.0, 146.9), turned to -20 degrees
- moved D29 12.5 mm to (167.5, 118.5)
- moved RE1 12.0 mm to (167.0, 126.5)
- moved S28 8.89 mm to (163.7, 155.9), turned to 160 degrees
- moved D25 5.83 mm to (104.0, 141.0)
- moved D26 5.83 mm to (123.0, 140.0)
- moved RE2 5.83 mm to (103.0, 149.8)
- moved S25 5.83 mm to (103.0, 151.0)
- moved S26 5.83 mm to (122.0, 150.0)
- moved D27 5.22 mm to (143.9, 141.1)
- moved S27 5.22 mm to (142.0, 151.0)
Other:
- board size 138.8 x 106.7 mm -> 138.8 x 113.9 mm
