File: evo56/GLP/ergogen/output/pcbs/left.kicad_pcb (KiCad board)
At the start: 2 copper layers, 138.8 x 113.9 mm, 68 parts

Commit message: yep
Parts:
- added JST1: , ceoloide:battery_connector_jst_ph_2, F.Cu at (170.6, 108.0)
- moved D29 3.60 mm to (167.5, 114.9)
- moved RE1 3.60 mm to (167.0, 122.9)
- moved D27 2.50 mm to (145.9, 142.6)
- moved S27 2.50 mm to (144.0, 152.5)
- moved D25 2.06 mm to (106.0, 141.5)
- moved D26 2.06 mm to (125.0, 140.5)
- moved RE2 2.06 mm to (105.0, 150.3)
- moved S25 2.06 mm to (105.0, 151.5)
- moved S26 2.06 mm to (124.0, 150.5)
- moved D28 1.48 mm to (167.1, 145.7), turned to -13 degrees
- moved PAD1 0.71 mm to (167.5, 66.5)
- moved S28 0.69 mm to (163.8, 155.2), turned to 167 degrees
Connections:
- PAD1 pad 2: BAT_RAW -> ON_P
Other:
- board size 138.8 x 113.9 mm -> 137.8 x 109.8 mm

Commit message: yep
Parts:
- moved ? 0.50 mm to (167.0, 70.5)
- moved CONN1 0.50 mm to (167.0, 75.5)
- moved D29 0.50 mm to (167.0, 114.9)
- moved DISP1 0.50 mm to (167.0, 83.5)
- moved MCU1 0.50 mm to (167.0, 81.5)
- moved PAD1 0.50 mm to (167.0, 66.5)
- moved RE1 0.50 mm to (166.5, 122.9)
Connections:
- MCU1 pad 10: col2 -> row2
- MCU1 pad 11: col3 -> row3
- MCU1 pad 12: col4 -> row4
- MCU1 pad 13: row5 -> col5
- MCU1 pad 14: row4 -> col4
- MCU1 pad 15: row3 -> col3
- MCU1 pad 16: row2 -> col2
- MCU1 pad 17: row1 -> col1
- MCU1 pad 18: row0 -> col0
- MCU1 pad 8: col0 -> row0
- MCU1 pad 9: col1 -> row1

Commit message: yep
Parts:
- added H3: , ceoloide:mounting_hole_plated, F.Cu at (175.0, 104.0)
- moved H1 89.5 mm to (72.0, 90.0)
- moved H2 15.2 mm to (160.0, 104.0)
- moved D13 4.50 mm to (107.0, 127.0)
- moved D14 4.50 mm to (107.0, 108.0)
- moved D15 4.50 mm to (107.0, 89.0)
- moved D16 4.50 mm to (107.0, 70.0)
- moved S13 4.50 mm to (107.0, 121.0)
- moved S14 4.50 mm to (107.0, 102.0)
- moved S15 4.50 mm to (107.0, 83.0)
- moved S16 4.50 mm to (107.0, 64.0)
- moved D10 3.50 mm to (88.0, 112.0)
- moved D11 3.50 mm to (88.0, 93.0)
- moved D12 3.50 mm to (88.0, 74.0)
- moved D9 3.50 mm to (88.0, 131.0)
- moved S10 3.50 mm to (88.0, 106.0)
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Other:
- board size 137.8 x 109.8 mm -> 137.8 x 112.1 mm

Commit message: yep
Parts:
- added H4: , ceoloide:mounting_hole_plated, F.Cu at (136.0, 111.0)
- added H5: , ceoloide:mounting_hole_plated, F.Cu at (157.4, 136.6)
- added H6: , ceoloide:mounting_hole_plated, F.Cu at (160.0, 104.0)
- added H7: , ceoloide:mounting_hole_plated, F.Cu at (175.0, 104.0)
- moved H2 100.8 mm to (60.0, 117.0)
- moved H3 49.8 mm to (136.0, 73.0)
- moved H1 16.3 mm to (60.0, 79.0)
- moved D28 2.15 mm to (168.4, 145.9), turned to -18 degrees
- moved S28 1.84 mm to (164.3, 155.1), turned to 162 degrees
- moved D25 1.00 mm to (105.0, 138.5)
- moved D26 1.00 mm to (124.0, 137.5)
- moved RE2 1.00 mm to (104.0, 147.3)
- moved S25 1.00 mm to (104.0, 148.5)
- moved S26 1.00 mm to (123.0, 147.5)
- moved D27 0.88 mm to (146.7, 139.8), turned to -10 degrees
- turned S27 to 170 degrees
Other:
- board size 137.8 x 112.1 mm -> 137.8 x 114.5 mm

Commit message: yep
Parts:
- moved D25 0.50 mm to (105.5, 138.5)
- moved D26 0.50 mm to (124.5, 137.5)
- moved D27 0.50 mm to (147.2, 139.8)
- moved D28 0.50 mm to (168.9, 145.9)
- moved H5 0.50 mm to (157.9, 136.6)
- moved RE2 0.50 mm to (104.5, 147.3)
- moved S25 0.50 mm to (104.5, 148.5)
- moved S26 0.50 mm to (123.5, 147.5)
- moved S27 0.50 mm to (144.5, 149.5)
- moved S28 0.50 mm to (164.8, 155.1)
Other:
- board size 137.8 x 114.5 mm -> 138.1 x 114.5 mm
- board text added: "imadam.xyz"
Changed lines of the file:
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@@
   (title_block
     (title "left")
-    (date "2025-04-11")
+    (date "2025-04-12")
     (rev "v1.0.0")
     (company "Unknown")
@@
   (footprint "ceoloide:switch_gateron_ks27_ks33"
     (layer "B.Cu")
-    (at 104 148.5 180)
+    (at 104.5 148.5 180)
     (property "Reference" "S25"
       (at 0 8.8 180)
@@
   (footprint "ceoloide:switch_gateron_ks27_ks33"
     (layer "B.Cu")
-    (at 123 147.5 180)
+    (at 123.5 147.5 180)
     (property "Reference" "S26"
       (at 0 8.8 180)
@@
   (footprint "ceoloide:switch_gateron_ks27_ks33"
     (layer "B.Cu")
-    (at 144 149.5 170)
+    (at 144.5 149.5 170)
     (property "Reference" "S27"
       (at 0 8.8 170)
@@
   (footprint "ceoloide:switch_gateron_ks27_ks33"
     (layer "B.Cu")
-    (at 164.3336665 155.1162272 162)
+    (at 164.8336665 155.1162272 162)
     (property "Reference" "S28"
       (at 0 8.8 162)
@@
     (footprint "ceoloide:diode_tht_sod123"
         (layer "B.Cu")
-        (at 105 138.5 0)
+        (at 105.5 138.5 0)
         (property "Reference" "D25"
             (at 0 0 0)
@@
     (footprint "ceoloide:diode_tht_sod123"
         (layer "B.Cu")
-        (at 124 137.5 0)
+        (at 124.5 137.5 0)
         (property "Reference" "D26"
             (at 0 0 0)
@@
     (footprint "ceoloide:diode_tht_sod123"
         (layer "B.Cu")
-        (at 146.7212895 139.8255706 -10)
+        (at 147.2212895 139.8255706 -10)
         (property "Reference" "D27"
             (at 0 0 -10)
@@
     (footprint "ceoloide:diode_tht_sod123"
         (layer "B.Cu")
-        (at 168.374893 145.914679 -18)
+        (at 168.874893 145.914679 -18)
         (property "Reference" "D28"
             (at 0 0 -18)
@@
   (footprint "ceoloide:rotary_encoder_ec11_ec12"
     (layer "F.Cu")
-    (at 104 147.3 0)
+    (at 104.5 147.3 0)
     (property "Reference" "RE2"
       (at 0 -8.5)
@@
     )
   )
+  (gr_text "imadam.xyz"
+    (at 123.5 152.5 -2.1)
+    (layer "F.SilkS" knockout)
+    (effects
+      (font
+        (size 2 2)
+        (thickness 1)
+      )
+    )
+  )
   (gr_text "Bottom"
-    (at 142.9581109 155.4088465 -10)
+    (at 143.4581109 155.4088465 -10)
     (layer "B.SilkS" knockout)
     (effects
@@
   (footprint "ceoloide:mounting_hole_plated"
     (layer "F.Cu")
-    (at 157.4376079 136.6380137 -10)
+    (at 157.9376079 136.6380137 -10)
     (property "Reference" "H5"
       (at 0 3 -10)
@@
 (gr_line (start 135.0527864 58.605572800000004) (end 135.9472136 60.394427199999996) (layer Edge.Cuts) (stroke (width 0.15) (type default)))
 (gr_line (start 137.736068 61.5) (end 175.25 61.5) (layer Edge.Cuts) (stroke (width 0.15) (type default)))
-(gr_line (start 177.25 147.46470212310305) (end 177.25 63.5) (layer Edge.Cuts) (stroke (width 0.15) (type default)))
-(gr_line (start 177.2487544998755 147.53527492662943) (end 177.12282001791831 151.10197839277316) (layer Edge.Cuts) (stroke (width 0.15) (type default)))
-(gr_line (start 177.0261785180427 151.64943958924675) (end 172.1782699905914 166.569767856388) (layer Edge.Cuts) (stroke (width 0.15) (type default)))
-(gr_line (start 169.6288008212167 167.8440683668649) (end 150.82689359286587 161.41204923834988) (layer Edge.Cuts) (stroke (width 0.15) (type default)))
-(gr_line (start 150.25253062349123 161.30571614882666) (end 114.50890967097112 160.00032538958962) (layer Edge.Cuts) (stroke (width 0.15) (type default)))
-(gr_line (start 114.49108746664122 159.9995948848473) (end 93.17243846297781 159.0305653846808) (layer Edge.Cuts) (stroke (width 0.15) (type default)))
-(gr_line (start 91.9828850673077 158.56907088942307) (end 77.98874008837211 146.90728340697677) (layer Edge.Cuts) (stroke (width 0.15) (type default)))
-(gr_line (start 76.86577629621794 146.44992970759614) (end 41.34259499215416 143.64546802569637) (layer Edge.Cuts) (stroke (width 0.15) (type default)))
+(gr_line (start 177.25 147.40672808811928) (end 177.25 63.5) (layer Edge.Cuts) (stroke (width 0.15) (type default)))
+(gr_line (start 177.25868069159966 147.59286649825185) (end 177.57446947958138 150.97119166858852) (layer Edge.Cuts) (stroke (width 0.15) (type default)))
+(gr_line (start 177.4852631711811 151.7753640787214) (end 172.67826999059136 166.56976785638813) (layer Edge.Cuts) (stroke (width 0.15) (type default)))
+(gr_line (start 170.12880082121674 167.84406836686492) (end 151.32689359286587 161.41204923834988) (layer Edge.Cuts) (stroke (width 0.15) (type default)))
+(gr_line (start 150.75253062349125 161.30571614882666) (end 115.00890967097482 160.00032538958976) (layer Edge.Cuts) (stroke (width 0.15) (type default)))
+(gr_line (start 114.99108746664493 159.9995948848475) (end 93.65460794576646 159.02975490662575) (layer Edge.Cuts) (stroke (width 0.15) (type default)))
+(gr_line (start 92.4899183406386 158.58864382309565) (end 77.98147922836091 146.88828970029107) (layer Edge.Cuts) (stroke (width 0.15) (type default)))
+(gr_line (start 76.883379226749 146.45131941263807) (end 41.34259499215416 143.6454680256964) (layer Edge.Cuts) (stroke (width 0.15) (type default)))
 (gr_arc (start 41.5 63.5) (mid 40.0857864 64.0857864) (end 39.5 65.5) (layer Edge.Cuts) (stroke (width 0.15) (type default)))
 (gr_arc (start 76.05848156666667 63.5) (mid 77.22790206666667 63.1224844) (end 77.95584816666667 62.1324556) (layer Edge.Cuts) (stroke (width 0.15) (type default)))
@@
 (gr_arc (start 135.9472136 60.3944272) (mid 136.68460579999999 61.2013016) (end 137.736068 61.5) (layer Edge.Cuts) (stroke (width 0.15) (type default)))
 (gr_arc (start 177.25 63.5) (mid 176.6642136 62.0857864) (end 175.25 61.5) (layer Edge.Cuts) (stroke (width 0.15) (type default)))
-(gr_arc (start 177.2487545 147.53527492310306) (mid 177.2496886 147.49999402310306) (end 177.25 147.46470212310305) (layer Edge.Cuts) (stroke (width 0.15) (type default)))
-(gr_arc (start 177.0261785180428 151.64943958924678) (mid 177.0936137180428 151.37908318924678) (end 177.1228200180428 151.1019783892468) (layer Edge.Cuts) (stroke (width 0.15) (type default)))
-(gr_arc (start 169.62880079059138 167.84406835638805) (mid 171.17034049059137 167.74071005638805) (end 172.1782699905914 166.56976785638804) (layer Edge.Cuts) (stroke (width 0.15) (type default)))
-(gr_arc (start 150.82689362349123 161.41204924882663) (mid 150.54361502349124 161.33780104882663) (end 150.25253062349125 161.30571624882663) (layer Edge.Cuts) (stroke (width 0.15) (type default)))
-(gr_arc (start 114.49108747097114 159.99959488958962) (mid 114.49999777097113 159.9999799895896) (end 114.50890967097114 160.00032538958962) (layer Edge.Cuts) (stroke (width 0.15) (type default)))
-(gr_arc (start 91.98288506730769 158.56907088942307) (mid 92.5398723673077 158.89722458942308) (end 93.1724384673077 159.0305653894231) (layer Edge.Cuts) (stroke (width 0.15) (type default)))
-(gr_arc (start 77.98874008837211 146.90728340697677) (mid 77.4627527883721 146.59145480697677) (end 76.8657762883721 146.44992970697675) (layer Edge.Cuts) (stroke (width 0.15) (type default)))
+(gr_arc (start 177.25 147.40672808811928) (mid 177.2521714 147.49989848811927) (end 177.2586807 147.59286648811928) (layer Edge.Cuts) (stroke (width 0.15) (type default)))
+(gr_arc (start 177.4852631711811 151.7753640787213) (mid 177.57095727118107 151.37783607872132) (end 177.57446947118106 150.9711916787213) (layer Edge.Cuts) (stroke (width 0.15) (type default)))
+(gr_arc (start 170.12880079059138 167.84406835638816) (mid 171.67034049059137 167.74071005638817) (end 172.6782699905914 166.56976785638815) (layer Edge.Cuts) (stroke (width 0.15) (type default)))
+(gr_arc (start 151.32689362349126 161.41204924882663) (mid 151.04361502349127 161.33780104882663) (end 150.75253062349128 161.30571624882663) (layer Edge.Cuts) (stroke (width 0.15) (type default)))
+(gr_arc (start 114.99108747097483 159.99959488958976) (mid 114.99999777097483 159.99997998958975) (end 115.00890967097483 160.00032538958976) (layer Edge.Cuts) (stroke (width 0.15) (type default)))
+(gr_arc (start 92.48991835009635 158.58864381136803) (mid 93.03705245009634 158.90216821136804) (end 93.65460795009635 159.02975491136803) (layer Edge.Cuts) (stroke (width 0.15) (type default)))
+(gr_arc (start 77.98147921890316 146.88828971201866) (mid 77.46544321890316 146.58684081201866) (end 76.88337921890316 146.45131941201865) (layer Edge.Cuts) (stroke (width 0.15) (type default)))
 (gr_arc (start 39.5 141.65167172631578) (mid 40.0311893 143.00909392631578) (end 41.342595 143.6454680263158) (layer Edge.Cuts) (stroke (width 0.15) (type default)))
 )
