File: evo56/GLP/ergogen/output/pcbs/left.kicad_pcb (KiCad board)
At the start: 2 copper layers, 138.1 x 114.5 mm, 74 parts

Commit message: yep
Parts:
- removed H6, H7: , ceoloide:mounting_hole_plated
- added H11: , ceoloide:mounting_hole_plated, F.Cu at (159.0, 110.0)
- added H12: , ceoloide:mounting_hole_plated, F.Cu at (175.0, 110.0)
- added kibuzzard-67FC4DE7: G***, kibuzzard-67FC4DE7, F.Cu at (124.2, 157.8)
- added kibuzzard-67FC4E9B: G***, kibuzzard-67FC4E9B, F.Cu at (60.6, 141.8)
- added kibuzzard-67FC4FAA: G***, kibuzzard-67FC4FAA, F.Cu at (166.5, 121.4)
- added kibuzzard-67FC4FC2: G***, kibuzzard-67FC4FC2, F.Cu at (163.6, 162.4)
- added kibuzzard-67FC4FD3: G***, kibuzzard-67FC4FD3, F.Cu at (166.3, 83.5)
- added kibuzzard-67FC4FE0: G***, kibuzzard-67FC4FE0, F.Cu at (168.3, 83.7)
- moved PWR1 5.00 mm to (175.5, 133.0), turned to 0 degrees
- moved RST1 5.00 mm to (175.0, 143.0)
- moved D27 1.41 mm to (148.2, 140.8)
- moved H5 1.41 mm to (158.9, 137.6)
- moved S28 1.41 mm to (165.8, 156.1)
- moved D25 1.41 mm to (106.5, 139.5)
- moved D26 1.41 mm to (125.5, 138.5)
- moved D28 1.41 mm to (169.9, 146.9)
- moved RE2 1.41 mm to (105.5, 148.3)
- moved S25 1.41 mm to (105.5, 149.5)
- moved S26 1.41 mm to (124.5, 148.5)
- moved S27 1.41 mm to (145.5, 150.5)
- moved D29 1.12 mm to (166.5, 113.4)
- moved ? 1.00 mm to (167.0, 69.0)
- moved CONN1 1.00 mm to (167.0, 74.0)
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Other:
- board size 138.1 x 114.5 mm -> 139.9 x 114.8 mm
- board text removed: "Battery"
- board text removed: "Bottom"
- board text removed: "Controller"
- board text removed: "Designed by imadam"
- board text removed: "Encoder"
- board text removed: "Left Side"
- board text removed: "imadam.xyz"
- board text removed: "← Power"
- board text removed: "← Reset"
