File: evo56/GLP/ergogen/output/pcbs/left.kicad_pcb (KiCad board)
At the start: 2 copper layers, 139.9 x 114.8 mm, 79 parts

Commit message: 40% > 50%
Parts:
- removed H10, H6, H7, H8, H9: , ceoloide:mounting_hole_plated
- added REF**: RollerEncoder_Panasonic_EVQWGD001, scroll:RollerEncoder_Panasonic_EVQWGD001, F.Cu at (166.8, 121.1)
- RE1, RE2: moved to B.Cu
Connections:
- D29 pad 1: row2 -> row4
- RE2 pad S1: col2 -> col1
- S25 pad 1: col2 -> col1
- S26 pad 1: col3 -> col2
- S27 pad 1: col4 -> col3
- S28 pad 1: col5 -> col4
Routing:
- net col1: track 0.00 -> 199.9 mm, vias 0 -> 3
- net GND: track 0.00 -> 189.5 mm, vias 0 -> 5
- net col2: track 0.00 -> 180.5 mm, vias 0 -> 3
- net row3: track 0.00 -> 171.3 mm, vias 0 -> 8
- net col0: track 0.00 -> 170.1 mm, vias 0 -> 1
- net col3: track 0.00 -> 167.6 mm, vias 0 -> 3
- net row2: track 0.00 -> 167.5 mm, vias 0 -> 10
- net col4: track 0.00 -> 152.7 mm, vias 0 -> 3
- net row1: track 0.00 -> 139.3 mm, vias 0 -> 10
- net row0: track 0.00 -> 138.4 mm, vias 0 -> 11
- net row4: track 0.00 -> 129.1 mm, vias 0 -> 9
- net ENCC: track 0.00 -> 103.2 mm, vias 0 -> 3
- net ON_P: track 0.00 -> 100.6 mm, vias 0 -> 4
- net col5: track 0.00 -> 98.9 mm, vias 0 -> 3
- net ENCD: track 0.00 -> 97.7 mm, vias 0 -> 2
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