File: evo56/GLP/ergogen/output/pcbs/right.kicad_pcb (KiCad board)
At the start: 2 copper layers, 139.9 x 114.8 mm, 79 parts

Commit message: 40% > 50%
Connections:
- D29 pad 1: row2 -> row4
- RE2 pad S1: col2 -> col1
- S25 pad 1: col2 -> col1
- S26 pad 1: col3 -> col2
- S27 pad 1: col4 -> col3
- S28 pad 1: col5 -> col4
Changed lines of the file:
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@@
   (title_block
     (title "right")
-    (date "2025-04-14")
+    (date "2025-04-18")
     (rev "v1.0.0")
     (company "Unknown")
@@
     (attr exclude_from_pos_files exclude_from_bom allow_soldermask_bridges)
     (pad "" thru_hole circle (at 0 0 -180) (size 5.6 5.6) (drill 5.1) (layers "*.Cu" "*.Mask") )
-    (pad "1" thru_hole circle (at -4.4 4.7 -180) (size 3.5 3.5) (drill 3) (layers "*.Cu" "*.Mask") (net 12 "col2"))
+    (pad "1" thru_hole circle (at -4.4 4.7 -180) (size 3.5 3.5) (drill 3) (layers "*.Cu" "*.Mask") (net 7 "col1"))
     (pad "2" thru_hole circle(at 2.6 5.75 -180) (size 3.5 3.5) (drill 3) (layers "*.Cu" "*.Mask") (net 32 "mirror_inner_cluster"))
-    (pad "1" smd roundrect (at -7.35 4.7 -180) (size 4 2.5) (layers "B.Cu") (roundrect_rratio 0.1) (net 12 "col2"))
+    (pad "1" smd roundrect (at -7.35 4.7 -180) (size 4 2.5) (layers "B.Cu") (roundrect_rratio 0.1) (net 7 "col1"))
     (pad "" smd roundrect (at -8.05 4.7 -180) (size 2.6 2.5) (layers "B.Paste" "B.Mask") (roundrect_rratio 0.1))
     (pad "2" smd roundrect (at 5.55 5.75 -180) (size 4 2.5) (layers "B.Cu") (roundrect_rratio 0.1) (net 32 "mirror_inner_cluster"))
@@
     (attr exclude_from_pos_files exclude_from_bom allow_soldermask_bridges)
     (pad "" thru_hole circle (at 0 0 -180) (size 5.6 5.6) (drill 5.1) (layers "*.Cu" "*.Mask") )
-    (pad "1" thru_hole circle (at -4.4 4.7 -180) (size 3.5 3.5) (drill 3) (layers "*.Cu" "*.Mask") (net 17 "col3"))
+    (pad "1" thru_hole circle (at -4.4 4.7 -180) (size 3.5 3.5) (drill 3) (layers "*.Cu" "*.Mask") (net 12 "col2"))
     (pad "2" thru_hole circle(at 2.6 5.75 -180) (size 3.5 3.5) (drill 3) (layers "*.Cu" "*.Mask") (net 33 "mirror_home_cluster"))
-    (pad "1" smd roundrect (at -7.35 4.7 -180) (size 4 2.5) (layers "B.Cu") (roundrect_rratio 0.1) (net 17 "col3"))
+    (pad "1" smd roundrect (at -7.35 4.7 -180) (size 4 2.5) (layers "B.Cu") (roundrect_rratio 0.1) (net 12 "col2"))
     (pad "" smd roundrect (at -8.05 4.7 -180) (size 2.6 2.5) (layers "B.Paste" "B.Mask") (roundrect_rratio 0.1))
     (pad "2" smd roundrect (at 5.55 5.75 -180) (size 4 2.5) (layers "B.Cu") (roundrect_rratio 0.1) (net 33 "mirror_home_cluster"))
@@
     (attr exclude_from_pos_files exclude_from_bom allow_soldermask_bridges)
     (pad "" thru_hole circle (at 0 0 -170) (size 5.6 5.6) (drill 5.1) (layers "*.Cu" "*.Mask") )
-    (pad "1" thru_hole circle (at -4.4 4.7 -170) (size 3.5 3.5) (drill 3) (layers "*.Cu" "*.Mask") (net 22 "col4"))
+    (pad "1" thru_hole circle (at -4.4 4.7 -170) (size 3.5 3.5) (drill 3) (layers "*.Cu" "*.Mask") (net 17 "col3"))
     (pad "2" thru_hole circle(at 2.6 5.75 -170) (size 3.5 3.5) (drill 3) (layers "*.Cu" "*.Mask") (net 34 "mirror_layer_cluster"))
-    (pad "1" smd roundrect (at -7.35 4.7 -170) (size 4 2.5) (layers "B.Cu") (roundrect_rratio 0.1) (net 22 "col4"))
+    (pad "1" smd roundrect (at -7.35 4.7 -170) (size 4 2.5) (layers "B.Cu") (roundrect_rratio 0.1) (net 17 "col3"))
     (pad "" smd roundrect (at -8.05 4.7 -170) (size 2.6 2.5) (layers "B.Paste" "B.Mask") (roundrect_rratio 0.1))
     (pad "2" smd roundrect (at 5.55 5.75 -170) (size 4 2.5) (layers "B.Cu") (roundrect_rratio 0.1) (net 34 "mirror_layer_cluster"))
@@
     (attr exclude_from_pos_files exclude_from_bom allow_soldermask_bridges)
     (pad "" thru_hole circle (at 0 0 -162) (size 5.6 5.6) (drill 5.1) (layers "*.Cu" "*.Mask") )
-    (pad "1" thru_hole circle (at -4.4 4.7 -162) (size 3.5 3.5) (drill 3) (layers "*.Cu" "*.Mask") (net 27 "col5"))
+    (pad "1" thru_hole circle (at -4.4 4.7 -162) (size 3.5 3.5) (drill 3) (layers "*.Cu" "*.Mask") (net 22 "col4"))
     (pad "2" thru_hole circle(at 2.6 5.75 -162) (size 3.5 3.5) (drill 3) (layers "*.Cu" "*.Mask") (net 35 "mirror_space_cluster"))
-    (pad "1" smd roundrect (at -7.35 4.7 -162) (size 4 2.5) (layers "B.Cu") (roundrect_rratio 0.1) (net 27 "col5"))
+    (pad "1" smd roundrect (at -7.35 4.7 -162) (size 4 2.5) (layers "B.Cu") (roundrect_rratio 0.1) (net 22 "col4"))
     (pad "" smd roundrect (at -8.05 4.7 -162) (size 2.6 2.5) (layers "B.Paste" "B.Mask") (roundrect_rratio 0.1))
     (pad "2" smd roundrect (at 5.55 5.75 -162) (size 4 2.5) (layers "B.Cu") (roundrect_rratio 0.1) (net 35 "mirror_space_cluster"))
@@
       (fp_line (start -0.35 0) (end -0.35 -0.55) (layer "B.SilkS") (stroke (width 0.1) (type solid)))
       (fp_line (start -0.75 0) (end -0.35 0) (layer "B.SilkS") (stroke (width 0.1) (type solid)))
-      (pad "1" smd rect (at -1.65 0 0) (size 0.9 1.2) (layers "B.Cu" "B.Paste" "B.Mask") (net 37 "row2"))
+      (pad "1" smd rect (at -1.65 0 0) (size 0.9 1.2) (layers "B.Cu" "B.Paste" "B.Mask") (net 40 "row4"))
       (pad "2" smd rect (at 1.65 0 0) (size 0.9 1.2) (layers "B.Cu" "B.Paste" "B.Mask") (net 41 "mirror_scrollwheel_enc"))
     )
@@
     (pad "B" thru_hole oval (at 0 7.5 0) (size 1.6 1.1) (drill oval 1 0.5) (layers "*.Cu" "F.Mask") (net 3 "GND"))
     (pad "C" thru_hole oval (at -2.5 7.5 0) (size 1.6 1.1) (drill oval 1 0.5) (layers "*.Cu" "F.Mask") (net 46 "ENCD"))
-    (pad "S1" thru_hole oval (at -2.5 -7 0) (size 1.6 1.1) (drill oval 1 0.5) (layers "*.Cu" "F.Mask") (net 12 "col2"))
+    (pad "S1" thru_hole oval (at -2.5 -7 0) (size 1.6 1.1) (drill oval 1 0.5) (layers "*.Cu" "F.Mask") (net 7 "col1"))
     (pad "S2" thru_hole oval (at 2.5 -7 0) (size 1.6 1.1) (drill oval 1 0.5) (layers "*.Cu" "F.Mask") (net 32 "mirror_inner_cluster"))
     (pad "" thru_hole roundrect
