File: evo56/GLP/PCB/Left/left.kicad_pcb (KiCad board)
At the start: 2 copper layers, 139.9 x 114.8 mm, 82 parts

Commit message: 40% > 50%
Parts:
- removed G***: LOGO, ok:qrcode
- removed the REF** at (166.8, 121.6)
- removed kibuzzard-67FD5276: G***, kibuzzard-67FD5276
- removed kibuzzard-67FD52AD: G***, kibuzzard-67FD52AD
- removed kibuzzard-67FD5311: G***, kibuzzard-67FD5311
- removed kibuzzard-67FD5341: G***, kibuzzard-67FD5341
- removed kibuzzard-67FD5486: G***, kibuzzard-67FD5486
- removed kibuzzard-67FD9A83: G***, kibuzzard-67FD9A83
- added REF**: RollerEncoder_Panasonic_EVQWGD001, scroll:RollerEncoder_Panasonic_EVQWGD001, F.Cu at (166.8, 121.1)
- RE1, RE2: moved to B.Cu
Connections:
- D29 pad 1: row2 -> row4
- RE2 pad S1: col2 -> col1
- S25 pad 1: col2 -> col1
- S26 pad 1: col3 -> col2
- S27 pad 1: col4 -> col3
- S28 pad 1: col5 -> col4
Routing:
- net col1: track 150.7 -> 199.9 mm, vias 4 -> 3
- net col5: track 144.2 -> 98.9 mm, vias 4 -> 3
- net col4: track 130.4 -> 152.7 mm, vias 4 -> 3
- net ON_P: track 80.9 -> 100.6 mm
- net col3: track 150.3 -> 167.6 mm, vias 4 -> 3
- net col2: track 169.6 -> 180.5 mm
- net BAT_GND: track 72.6 -> 83.4 mm, vias 3 -> 0
- net row2: track 156.9 -> 167.5 mm, vias 14 -> 10
- net ENCD: track 107.1 -> 97.7 mm, vias 5 -> 2
- net GND: track 197.0 -> 189.5 mm, vias 8 -> 5
- net row4: track 124.1 -> 129.1 mm, vias 8 -> 9
- net RST: track 93.4 -> 89.7 mm, vias 2 -> 6
- net ENCB: track 46.7 -> 50.4 mm, vias 2 -> 3
- net scrollwheel_enc: track 23.5 -> 19.8 mm, vias 4 -> 1
- net inner_bottom: track 14.8 -> 18.4 mm
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- removed copper zone on B.Cu, net (none)
- removed copper zone on F.Cu, net (none)

Commit message: finish right glp pcb
Parts:
- added Board_0-G***: LOGO, ok:qrcode, F.Cu at (87.8, 146.6)
- added Board_0-kibuzzard-67FD5276: G***, kibuzzard-67FD5276, F.Cu at (61.6, 141.4)
- added Board_0-kibuzzard-67FD52AD: G***, kibuzzard-67FD52AD, F.Cu at (125.0, 158.0)
- added Board_0-kibuzzard-67FD5311: G***, kibuzzard-67FD5311, F.Cu at (166.0, 81.2)
- added Board_0-kibuzzard-67FD5341: G***, kibuzzard-67FD5341, F.Cu at (167.8, 81.2)
- added Board_0-kibuzzard-67FD5486: G***, kibuzzard-67FD5486, F.Cu at (167.8, 121.4)
- added Board_0-kibuzzard-67FD9A83: G***, kibuzzard-67FD9A83, F.Cu at (164.8, 162.8)
- RE1, RE2: moved to F.Cu
- turned RE1 to 90 degrees
- turned RE2 to 180 degrees
Routing:
- net ENCA: track 53.4 -> 46.9 mm
- net ENCD: track 97.7 -> 92.7 mm
- net scrollwheel_enc: track 19.8 -> 15.3 mm, vias 1 -> 3
- net RST: track 89.7 -> 85.4 mm
- net col5: track 98.9 -> 102.9 mm
- net ENCC: track 103.2 -> 106.5 mm, vias 3 -> 2
- net ENCB: track 50.4 -> 52.8 mm
- net inner_cluster: track 12.3 -> 10.8 mm
- net row3: track 171.3 -> 171.5 mm, vias 8 -> 10
- added copper zone on B.Cu, net (none)
- added copper zone on F.Cu, net (none)
