File: evo56/GLP/PCB/Right/right.kicad_pcb (KiCad board)
At the start: 2 copper layers, 139.9 x 114.8 mm, 79 parts

Commit message: yep
Parts:
- moved D1 285.0 mm to (335.0, 137.0)
- moved D2 285.0 mm to (335.0, 118.0)
- moved D3 285.0 mm to (335.0, 99.0)
- moved D4 285.0 mm to (335.0, 80.0)
- moved S1 285.0 mm to (335.0, 131.0)
- moved S2 285.0 mm to (335.0, 112.0)
- moved S3 285.0 mm to (335.0, 93.0)
- moved S4 285.0 mm to (335.0, 74.0)
- moved D5 247.0 mm to (316.0, 137.0)
- moved D6 247.0 mm to (316.0, 118.0)
- moved D7 247.0 mm to (316.0, 99.0)
- moved D8 247.0 mm to (316.0, 80.0)
- moved S5 247.0 mm to (316.0, 131.0)
- moved S6 247.0 mm to (316.0, 112.0)
- moved S7 247.0 mm to (316.0, 93.0)
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Connections:
- net home_cluster renamed mirror_home_cluster
- net index_bottom renamed mirror_index_bottom
- net index_home renamed mirror_index_home
- net index_num renamed mirror_index_num
- net index_top renamed mirror_index_top
- net inner_bottom renamed mirror_inner_bottom
- net inner_cluster renamed mirror_inner_cluster
- net inner_home renamed mirror_inner_home
- net inner_num renamed mirror_inner_num
- net inner_top renamed mirror_inner_top
- net layer_cluster renamed mirror_layer_cluster
- net middle_bottom renamed mirror_middle_bottom
- net middle_home renamed mirror_middle_home
- net middle_num renamed mirror_middle_num
- net middle_top renamed mirror_middle_top
- net outer_bottom renamed mirror_outer_bottom
- net outer_home renamed mirror_outer_home
- net outer_num renamed mirror_outer_num
- net outer_top renamed mirror_outer_top
- net pinky_bottom renamed mirror_pinky_bottom
- net pinky_home renamed mirror_pinky_home
- net pinky_num renamed mirror_pinky_num
- net pinky_top renamed mirror_pinky_top
- net ring_bottom renamed mirror_ring_bottom
- net ring_home renamed mirror_ring_home
- net ring_num renamed mirror_ring_num
- net ring_top renamed mirror_ring_top
- net space_cluster renamed mirror_space_cluster
- D29 pad 2: scrollwheel_enc -> mirror_scrollwheel_enc
Other:
- outline, holes or cut-outs redrawn

Commit message: yep
Parts:
- removed H1, H2, H3, H4, H5: , ceoloide:mounting_hole_plated
- added G***: LOGO, ok:qrcode, F.Cu at (295.6, 148.0)
- added G***: LOGO, asdf:merc, B.Cu at (220.8, 161.6)
- added REF**: RollerEncoder_Panasonic_EVQWGD001, ok:RollerEncoder_Panasonic_EVQWGD001, F.Cu at (219.2, 121.0)
- added kibuzzard-67FD5311: G***, kibuzzard-67FD5311, F.Cu at (216.6, 81.4)
- added kibuzzard-67FD5341: G***, kibuzzard-67FD5341, F.Cu at (218.4, 81.4)
- added kibuzzard-67FD5486: G***, kibuzzard-67FD5486, F.Cu at (219.6, 121.0)
- added kibuzzard-67FD9A7A: G***, kibuzzard-67FD9A7A, F.Cu at (220.6, 163.4)
- added kibuzzard-67FD9A9C: G***, kibuzzard-67FD9A9C, F.Cu at (253.6, 159.4)
- added kibuzzard-67FD9ADD: G***, kibuzzard-67FD9ADD, F.Cu at (324.8, 140.8)
- turned PWR1 to 180 degrees
Connections:
- D29 pad 2: mirror_scrollwheel_enc -> scrollwheel_enc
Routing:
- net col2: track 0.00 -> 207.0 mm, vias 0 -> 2
- net col0: track 0.00 -> 199.3 mm
- net GND: track 0.00 -> 194.2 mm, vias 0 -> 1
- net col5: track 0.00 -> 188.7 mm, vias 0 -> 4
- net col1: track 0.00 -> 187.6 mm, vias 0 -> 4
- net col4: track 0.00 -> 179.4 mm, vias 0 -> 2
- net col3: track 0.00 -> 178.7 mm, vias 0 -> 2
- net row2: track 0.00 -> 169.1 mm, vias 0 -> 15
- net row3: track 0.00 -> 155.1 mm, vias 0 -> 9
- net row4: track 0.00 -> 141.4 mm, vias 0 -> 14
- net ENCC: track 0.00 -> 128.3 mm, vias 0 -> 2
- net ENCD: track 0.00 -> 122.0 mm, vias 0 -> 3
- net row0: track 0.00 -> 120.8 mm, vias 0 -> 11
- net row1: track 0.00 -> 120.6 mm, vias 0 -> 11
- net ON_P: track 0.00 -> 80.5 mm, vias 0 -> 6
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- added copper zone on B.Cu, net (none)
- added copper zone on F.Cu, net (none)
